File: Kicad/bs_sensor_stm32/bs_sensor_stm32/bs_sensor_stm32.kicad_pcb (KiCad board)
At the start: 2 copper layers, 1 part, among them U1 NRF24L01_Breakout

Commit message: 01.03.2022
Parts:
- added C1: 22p, Capacitor_SMD:C_0805_2012Metric, B.Cu at (160.8, 100.8)
- added C2: 100n, Capacitor_SMD:C_0805_2012Metric, B.Cu at (177.8, 106.4)
- added C3: 10u, Capacitor_SMD:C_0805_2012Metric, B.Cu at (177.8, 108.5)
- added C4: 22p, Capacitor_SMD:C_0805_2012Metric, B.Cu at (164.3, 100.8)
- added C5: 100n, Capacitor_SMD:C_0805_2012Metric, B.Cu at (166.4, 106.4)
- added C6: 100n, Capacitor_SMD:C_0805_2012Metric, B.Cu at (166.4, 110.0)
- added D1: 1N4148W, Diode_SMD:D_SOD-123, F.Cu at (169.7, 107.4)
- added J1: Conn_01x02, Connector_PinHeader_2.54mm:PinHeader_1x02_P2.54mm_Vertical, F.Cu at (164.1, 113.3)
- added J2: Conn_01x04, Connector_PinHeader_2.54mm:PinHeader_1x04_P2.54mm_Vertical, F.Cu at (170.4, 113.3)
- added J3: Conn_01x04, Connector_PinHeader_2.54mm:PinHeader_1x04_P2.54mm_Vertical, F.Cu at (170.4, 101.6)
- added J4: Conn_01x04, Connector_PinHeader_2.54mm:PinHeader_1x04_P2.54mm_Vertical, F.Cu at (152.7, 113.3)
- added JP1: SolderJumper_2_Open, Jumper:SolderJumper-2_P1.3mm_Open_RoundedPad1.0x1.5mm, F.Cu at (158.2, 108.7)
- added JP2: SolderJumper_2_Open, Jumper:SolderJumper-2_P1.3mm_Open_RoundedPad1.0x1.5mm, F.Cu at (164.3, 108.7)
- added R1: 10k, Resistor_SMD:R_0805_2012Metric, F.Cu at (163.1, 106.4)
- added R2: 620, Resistor_SMD:R_0603_1608Metric, F.Cu at (158.0, 106.4)
- added R3: 10k, Resistor_SMD:R_0805_2012Metric, B.Cu at (172.2, 106.4)
- added R4: 4,7k, Resistor_SMD:R_0805_2012Metric, B.Cu at (172.2, 108.5)
- added U2: AMS1117-3.3, Package_TO_SOT_SMD:SOT-223-3_TabPin2, F.Cu at (175.5, 107.4)
- added U3: STM32F030F4Px, Package_SO:TSSOP-20_4.4x6.5mm_P0.65mm, B.Cu at (160.5, 107.4)
- added Y1: 16MHz, Crystal:Crystal_HC49-U_Vertical, F.Cu at (160.0, 102.6)
- moved U1 0.22 mm to (152.4, 101.8)
Connections:
- U1 pad 1: unconnected-(U1-Pad1) -> GND
- U1 pad 2: unconnected-(U1-Pad2) -> +3V3
- U1 pad 3: unconnected-(U1-Pad3) -> Net-(U1-Pad3)
- U1 pad 4: unconnected-(U1-Pad4) -> Net-(U1-Pad4)
- U1 pad 5: unconnected-(U1-Pad5) -> Net-(U1-Pad5)
- U1 pad 6: unconnected-(U1-Pad6) -> Net-(U1-Pad6)
- U1 pad 7: unconnected-(U1-Pad7) -> Net-(U1-Pad7)
- U1 pad 8: unconnected-(U1-Pad8) -> Net-(U1-Pad8)
Routing:
- net +3V3: track 0.00 -> 79.4 mm
- net Net-(C4-Pad1): track 0.00 -> 14.5 mm
- net Net-(U1-Pad6): track 0.00 -> 11.0 mm
- net Net-(U1-Pad3): track 0.00 -> 9.72 mm
- net Net-(D1-Pad2): track 0.00 -> 5.45 mm
- net Net-(D1-Pad1): track 0.00 -> 5.44 mm
- net Net-(U1-Pad8): track 0.00 -> 5.17 mm
- net Net-(C1-Pad2): track 0.00 -> 4.59 mm
- added copper zone on B.Cu, net GND
- added copper zone on F.Cu, net GND
Other:
- board text added: "+"
- board text added: "-"
- board text added: "a0"
- board text added: "a1"
- board text added: "a10"
- board text added: "a9"
- board text added: "b1"
- board text added: "bs_sens"
- board text added: "clk"
- board text added: "dio"
- board text added: "gnd"
- board text added: "nrf24l01+"
- board text added: "vcc"

Commit message: 01.03.2022
Parts:
- moved C6 0.25 mm to (166.4, 110.2)
- turned JP2 to 0 degrees
Routing:
- net GND: track 0.00 -> 60.4 mm, vias 0 -> 16
- net Net-(J2-Pad2): track 0.00 -> 42.0 mm
- net Net-(C6-Pad1): track 0.00 -> 32.8 mm, vias 0 -> 2
- net Net-(J3-Pad2): track 0.00 -> 30.6 mm
- net Net-(J3-Pad3): track 0.00 -> 24.1 mm, vias 0 -> 2
- net Net-(U1-Pad7): track 0.00 -> 20.2 mm, vias 0 -> 1
- net Net-(J2-Pad4): track 0.00 -> 18.3 mm, vias 0 -> 1
- net Net-(J4-Pad3): track 0.00 -> 16.8 mm, vias 0 -> 1
- net Net-(J2-Pad3): track 0.00 -> 16.7 mm, vias 0 -> 1
- net Net-(R2-Pad2): track 0.00 -> 14.5 mm, vias 0 -> 3
- net Net-(J4-Pad2): track 0.00 -> 14.3 mm, vias 0 -> 1
- net +3V3: track 79.4 -> 93.6 mm, vias 0 -> 1
- net Net-(U1-Pad5): track 0.00 -> 14.0 mm, vias 0 -> 1
- net Net-(JP1-Pad2): track 0.00 -> 11.1 mm
- net Net-(C1-Pad2): track 4.59 -> 12.3 mm, vias 0 -> 2
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
Commit message: 05.03.2022
Parts:
- JP1, JP2: footprint Jumper:SolderJumper-2_P1.3mm_Open_RoundedPad1.0x1.5mm -> Jumper:SolderJumper-2_P1.3mm_Open_TrianglePad1.0x1.5mm
- moved JP2 0.51 mm to (164.3, 109.2)
Routing:
- net GND: track 60.4 -> 65.0 mm
- net Net-(JP2-Pad2): track 6.84 -> 7.87 mm
- net Net-(J4-Pad3): track 16.8 -> 16.2 mm
- net Net-(J3-Pad3): track 24.1 -> 24.7 mm
Other:
- board outline added: 29.5 x 15.7 mm

Commit message: 07.09.2022
Routing:
- net +3V3: track 93.9 -> 93.0 mm
- net Net-(U1-Pad6): track 14.7 -> 14.0 mm
- net Net-(JP2-Pad2): track 7.87 -> 7.33 mm
Other:
- board text removed: "nrf24l01+"
Changed lines of the file:
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@@
     (property "Sheetname" "")
     (attr through_hole)
-    (fp_text reference "J2" (at 1.27 -1.016 180) (layer "F.SilkS")
+    (fp_text reference "J2" (at 1.778 -1.016 180) (layer "F.SilkS")
       (effects (font (size 1 1) (thickness 0.15)))
     )
@@
     (property "Sheetname" "")
     (attr through_hole)
-    (fp_text reference "J4" (at 1.27 -1.026 180) (layer "F.SilkS")
+    (fp_text reference "J4" (at 1.524 -1.026 180) (layer "F.SilkS")
       (effects (font (size 1 1) (thickness 0.15)))
     )
@@
     (effects (font (size 1 1) (thickness 0.15)) (justify mirror))
   )
-  (gr_text "nrf24l01+" (at 153.67 105.918 90) (layer "B.SilkS")
-    (effects (font (size 1 1) (thickness 0.15)) (justify mirror))
-  )
   (gr_text "vcc" (at 169.672 103.886 90) (layer "B.SilkS")
     (effects (font (size 1 1) (thickness 0.15)) (justify mirror))
@@
   (segment (start 168.402 113.284) (end 168.148 113.03) (width 0.5) (layer "B.Cu") (net 1))
   (segment (start 166.624011 102.142312) (end 166.624011 103.378011) (width 0.5) (layer "B.Cu") (net 1))
-  (segment (start 163.3905 107.117) (end 163.4615 107.188) (width 0.25) (layer "B.Cu") (net 1))
   (segment (start 167.110987 105.09752) (end 167.69848 105.09752) (width 0.25) (layer "B.Cu") (net 1))
   (segment (start 167.69848 105.09752) (end 168.656 104.14) (width 0.25) (layer "B.Cu") (net 1))
@@
   (segment (start 175.164489 103.942489) (end 173.538489 103.942489) (width 0.5) (layer "F.Cu") (net 3))
   (segment (start 153.67 100.584) (end 154.894 101.808) (width 0.5) (layer "F.Cu") (net 3))
-  (segment (start 154.894 101.817) (end 154.894 102.156047) (width 0.5) (layer "F.Cu") (net 3))
   (segment (start 166.78012 103.036489) (end 166.282489 103.53412) (width 0.5) (layer "F.Cu") (net 3))
   (segment (start 151.142489 100.605489) (end 151.163978 100.584) (width 0.5) (layer "F.Cu") (net 3))
@@
   (segment (start 166.965511 103.036489) (end 166.78012 103.036489) (width 0.5) (layer "F.Cu") (net 3))
   (segment (start 156.718 100.076) (end 168.91 100.076) (width 0.5) (layer "F.Cu") (net 3))
-  (segment (start 152.664 113.284) (end 153.162 113.284) (width 0.5) (layer "F.Cu") (net 3))
   (segment (start 171.733511 102.899511) (end 170.434 101.6) (width 0.5) (layer "F.Cu") (net 3))
   (segment (start 166.282489 103.719511) (end 165.936489 104.065511) (width 0.5) (layer "F.Cu") (net 3))
@@
   (segment (start 178.664 107.442) (end 175.164489 103.942489) (width 0.5) (layer "F.Cu") (net 3))
   (segment (start 172.495511 102.899511) (end 171.733511 102.899511) (width 0.5) (layer "F.Cu") (net 3))
-  (segment (start 154.894 101.817) (end 154.977 101.817) (width 0.5) (layer "F.Cu") (net 3))
   (via (at 174.498 107.442) (size 0.8) (drill 0.4) (layers "F.Cu" "B.Cu") (free) (net 3))
   (segment (start 174.498 107.442) (end 174.1405 107.442) (width 0.5) (layer "B.Cu") (net 3))
@@
   (segment (start 162.1555 106.426) (end 161.430989 107.150511) (width 0.25) (layer "F.Cu") (net 14))
   (segment (start 160.368609 109.205204) (end 160.368609 109.80541) (width 0.25) (layer "F.Cu") (net 14))
-  (segment (start 164.988 108.712) (end 164.988 109.145) (width 0.25) (layer "F.Cu") (net 15))
   (segment (start 166.37 109.22) (end 167.64 107.95) (width 0.25) (layer "F.Cu") (net 15))
-  (segment (start 164.988 109.145) (end 165.063 109.22) (width 0.25) (layer "F.Cu") (net 15))
   (segment (start 165.063 109.22) (end 166.37 109.22) (width 0.25) (layer "F.Cu") (net 15))
   (via (at 167.64 107.95) (size 0.8) (drill 0.4) (layers "F.Cu" "B.Cu") (free) (net 15))
@@
   (segment (start 159.474511 104.131397) (end 159.474511 105.372511) (width 0.25) (layer "B.Cu") (net 20))
   (segment (start 154.894 105.950639) (end 157.154119 103.69052) (width 0.25) (layer "B.Cu") (net 20))
-  (segment (start 162.661 105.817) (end 163.3905 105.817) (width 0.25) (layer "B.Cu") (net 20))
   (segment (start 154.894 106.897) (end 154.894 105.950639) (width 0.25) (layer "B.Cu") (net 20))
   (segment (start 163.3905 105.817) (end 161.645 105.817) (width 0.25) (layer "B.Cu") (net 20))
