File: Kicad/bs_sensor_nuvoton/bs_sensor_nuvoton/bs_sensor_nuvoton.kicad_pcb (KiCad board)
At the start: 2 copper layers, 29.5 x 15.7 mm, 22 parts, among them J1 Conn_01x02, J2 Conn_01x04, J3 Conn_01x04, J4 Conn_01x04, U1 NRF24L01_Breakout, U2 AMS1117-3.3, U3 STM32F030F4Px, U4 N76E003AT20, Y1 16MHz

Commit message: 07.09.2022
Parts:
- removed C1, C4: 22p, Capacitor_SMD:C_0805_2012Metric
- removed R1: 10k, Resistor_SMD:R_0805_2012Metric
- removed R2: 620, Resistor_SMD:R_0603_1608Metric
- removed U3: STM32F030F4Px, Package_SO:TSSOP-20_4.4x6.5mm_P0.65mm
- removed Y1: 16MHz, Crystal:Crystal_HC49-U_Vertical
- added J5: Conn_01x05, Connector_PinHeader_2.54mm:PinHeader_1x05_P2.54mm_Vertical, F.Cu at (141.0, 90.2)
- added JP3: SolderJumper_2_Open, Jumper:SolderJumper-2_P1.3mm_Open_TrianglePad1.0x1.5mm, B.Cu at (147.1, 81.5)
- C2, C3, R3: moved to F.Cu
- C6: value 100n -> 10u; moved to F.Cu
- J3: value Conn_01x04 -> Conn_01x02; footprint Connector_PinHeader_2.54mm:PinHeader_1x04_P2.54mm_Vertical -> Connector_PinHeader_2.54mm:PinHeader_1x02_P2.54mm_Vertical
- J4: value Conn_01x04 -> Conn_01x07; footprint Connector_PinHeader_2.54mm:PinHeader_1x04_P2.54mm_Vertical -> Connector_PinHeader_2.54mm:PinHeader_1x07_P2.54mm_Vertical
- JP1, JP2, U4: moved to B.Cu
- moved U4 58.3 mm to (137.4, 84.3), turned to -90 degrees
- moved J2 47.0 mm to (129.6, 90.2)
- moved C3 44.9 mm to (140.7, 83.1), turned to 180 degrees
- moved C2 42.8 mm to (140.7, 85.1), turned to 180 degrees
- moved R3 41.0 mm to (137.2, 85.1), turned to 0 degrees
- moved C6 39.9 mm to (137.2, 83.1)
- moved J4 38.9 mm to (135.4, 78.5)
- moved R4 38.3 mm to (144.3, 82.3), turned to 90 degrees
- moved U2 36.3 mm to (147.3, 84.6), turned to 180 degrees
- moved U1 32.7 mm to (129.2, 78.7)
- moved JP2 30.5 mm to (147.1, 84.1), turned to 180 degrees
- moved C5 30.2 mm to (144.3, 85.9), turned to -90 degrees
- moved J3 27.8 mm to (154.9, 78.5), turned to 0 degrees
- moved D1 27.7 mm to (154.4, 84.3), turned to 0 degrees
- moved J1 24.9 mm to (154.9, 90.2), turned to 180 degrees
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Connections:
- J3 pad 1: +3V3 -> Net-(J3-Pad1)
- J4 pad 4: GND -> Net-(J4-Pad4)
- JP1 pad 1: GND -> Net-(JP1-Pad1)
- JP1 pad 2: Net-(JP1-Pad2) -> Net-(J4-Pad3)
- JP2 pad 1: Net-(J4-Pad3) -> Net-(J5-Pad2)
- U1 pad 4: Net-(U1-Pad4) -> Net-(JP1-Pad1)
- U4 pad 1: unconnected-(U4-Pad1) -> Net-(J5-Pad3)
- U4 pad 10: unconnected-(U4-Pad10) -> Net-(J2-Pad4)
- U4 pad 11: unconnected-(U4-Pad11) -> Net-(J3-Pad2)
- U4 pad 12: unconnected-(U4-Pad12) -> Net-(J3-Pad1)
- U4 pad 13: unconnected-(U4-Pad13) -> Net-(J2-Pad2)
- U4 pad 14: unconnected-(U4-Pad14) -> Net-(J2-Pad3)
- U4 pad 15: unconnected-(U4-Pad15) -> Net-(U1-Pad5)
- U4 pad 16: unconnected-(U4-Pad16) -> Net-(U1-Pad6)
- U4 pad 17: unconnected-(U4-Pad17) -> Net-(U1-Pad7)
- U4 pad 18: unconnected-(U4-Pad18) -> Net-(J4-Pad3)
- U4 pad 19: unconnected-(U4-Pad19) -> Net-(U1-Pad3)
- U4 pad 2: unconnected-(U4-Pad2) -> Net-(J4-Pad7)
- U4 pad 20: unconnected-(U4-Pad20) -> Net-(J5-Pad2)
- U4 pad 3: unconnected-(U4-Pad3) -> Net-(J4-Pad6)
- U4 pad 4: unconnected-(U4-Pad4) -> Net-(J4-Pad4)
- U4 pad 5: unconnected-(U4-Pad5) -> Net-(U1-Pad8)
- U4 pad 6: unconnected-(U4-Pad6) -> Net-(J5-Pad4)
- U4 pad 7: unconnected-(U4-Pad7) -> GND
- U4 pad 8: unconnected-(U4-Pad8) -> Net-(J4-Pad2)
- U4 pad 9: unconnected-(U4-Pad9) -> +3V3
Routing:
- net +3V3: track 93.9 -> 41.5 mm, vias 1 -> 3
- net GND: track 65.0 -> 108.2 mm, vias 16 -> 8
- net Net-(J5-Pad3): track 0.00 -> 35.9 mm, vias 0 -> 1
- net Net-(J4-Pad6): track 0.00 -> 34.6 mm, vias 0 -> 2
- net Net-(J3-Pad1): track 0.00 -> 34.1 mm
- net Net-(J5-Pad4): track 0.00 -> 32.8 mm, vias 0 -> 1
- net Net-(J2-Pad2): track 42.4 -> 11.0 mm
- net Net-(J5-Pad2): track 0.00 -> 28.7 mm, vias 0 -> 2
- net Net-(J4-Pad7): track 0.00 -> 26.8 mm, vias 0 -> 2
- net Net-(J3-Pad3): track 24.7 -> 0.00 mm, vias 2 -> 0
- net Net-(JP1-Pad1): track 0.00 -> 21.6 mm
- net Net-(J4-Pad3): track 16.2 -> 36.7 mm, vias 1 -> 2
- net Net-(J4-Pad4): track 0.00 -> 20.1 mm, vias 0 -> 1
- net Net-(C4-Pad1): track 16.9 -> 0.00 mm, vias 1 -> 0
- net Net-(R2-Pad2): track 14.5 -> 0.00 mm, vias 3 -> 0
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Other:
- board text added: "0.4"
- board text added: "0.5"
- board text added: "1.1"
- board text added: "1.2"
- board text added: "1.5"
- board text added: "1.7"
- board text added: "bs sens"
- board text added: "dat"
- board text added: "rst"
- board text added: "rx"
- board text added: "scl"
- board text added: "sda"
- board text added: "tx"
- board text removed: "a0"
- board text removed: "a1"
- board text removed: "a10"
- board text removed: "a9"
- board text removed: "b1"
- board text removed: "bs_sens"
- board text removed: "dio"
- board text removed: "gnd"
- board text removed: "nrf24l01+"
- board text removed: "vcc"
