File: 433 MHz/TX_tiny10/TX_tiny10.kicad_pcb (KiCad board)
At the start: 2 copper layers, 3 parts, among them U1 ATtiny10-TS

Commit message: 21.06.2022
Parts:
- added SW1: SW_Push_DPDT, Button_Switch_THT:SW_Push_2P2T_Toggle_CK_PVA2xxH3xxxxxxV2, F.Cu at (160.0, 66.0)
Connections:
- BT1 pad 1: +3V3 -> Net-(BT1-Pad1)
Changed lines of the file:
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@@
   (net 5 "unconnected-(U1-Pad4)")
   (net 6 "unconnected-(U1-Pad6)")
+  (net 7 "Net-(BT1-Pad1)")
+  (net 8 "unconnected-(SW1-Pad3)")
+  (net 9 "unconnected-(SW1-Pad4)")
+  (net 10 "unconnected-(SW1-Pad5)")
+  (net 11 "unconnected-(SW1-Pad6)")
   (footprint "Package_TO_SOT_SMD:SOT-23-6" (layer "F.Cu")
     (at 149.835 73.405)
@@
       (net 6 "unconnected-(U1-Pad6)") (pinfunction "~{RESET}/PB3") (pintype "bidirectional"))
     (model "${KICAD6_3DMODEL_DIR}/Package_TO_SOT_SMD.3dshapes/SOT-23-6.wrl"
+      (offset (xyz 0 0 0))
+      (scale (xyz 1 1 1))
+      (rotate (xyz 0 0 0))
+    )
+  )
+  (footprint "Button_Switch_THT:SW_Push_2P2T_Toggle_CK_PVA2xxH3xxxxxxV2" (layer "F.Cu")
+    (at 160.02 66.04)
+    (descr "momentary / push-push button, h=20.5mm C&K PVA2 https://www.ckswitches.com/media/1343/pva.pdf")
+    (tags "tact sw push PVA2 DPDT")
+    (property "Sheetfile" "TX_tiny10.kicad_sch")
+    (property "Sheetname" "")
+    (attr through_hole)
+    (fp_text reference "SW1" (at 2.5 -2.75) (layer "F.SilkS")
+      (effects (font (size 1 1) (thickness 0.15)))
+    )
+    (fp_text value "SW_Push_DPDT" (at 2.5 9) (layer "F.Fab")
+      (effects (font (size 1 1) (thickness 0.15)))
+    )
+    (fp_text user "${REFERENCE}" (at 2.5 3) (layer "F.Fab")
+      (effects (font (size 1 1) (thickness 0.15)))
+    )
+    (fp_line (start -2.52 7.72) (end -2.52 -1.72) (layer "F.SilkS") (width 0.12))
+    (fp_line (start 4.1 4.6) (end 0.8 4.6) (layer "F.SilkS") (width 0.12))
+    (fp_line (start 0.8 1.3) (end 0.8 4.6) (layer "F.SilkS") (width 0.12))
+    (fp_line (start 4.1 1.3) (end 4.1 4.6) (layer "F.SilkS") (width 0.12))
+    (fp_line (start 4.1 1.3) (end 0.8 1.3) (layer "F.SilkS") (width 0.12))
+    (fp_line (start 7.52 7.72) (end -2.52 7.72) (layer "F.SilkS") (width 0.12))
+    (fp_line (start -1.77 -1.97) (end -2.77 -1.97) (layer "F.SilkS") (width 0.12))
+    (fp_line (start 7.52 7.72) (end 7.52 -1.72) (layer "F.SilkS") (width 0.12))
+    (fp_line (start -2.77 -0.97) (end -2.77 -1.97) (layer "F.SilkS") (width 0.12))
+    (fp_line (start 7.52 -1.72) (end -2.52 -1.72) (layer "F.SilkS") (width 0.12))
+    (fp_line (start -2.65 -1.85) (end 7.65 -1.85) (layer "F.CrtYd") (width 0.05))
+    (fp_line (start 7.65 -1.85) (end 7.65 7.85) (layer "F.CrtYd") (width 0.05))
+    (fp_line (start -2.65 7.85) (end 7.65 7.85) (layer "F.CrtYd") (width 0.05))
+    (fp_line (start -2.65 7.85) (end -2.65 -1.85) (layer "F.CrtYd") (width 0.05))
+    (fp_line (start 7.4 -1.6) (end 7.4 7.6) (layer "F.Fab") (width 0.1))
+    (fp_line (start -2.4 -0.6) (end -1.4 -1.6) (layer "F.Fab") (width 0.1))
+    (fp_line (start 7.4 7.6) (end -2.4 7.6) (layer "F.Fab") (width 0.1))
+    (fp_line (start -2.4 7.6) (end -2.4 -0.6) (layer "F.Fab") (width 0.1))
+    (fp_line (start -1.4 -1.6) (end 7.4 -1.6) (layer "F.Fab") (width 0.1))
+    (pad "1" thru_hole rect (at 0 0) (size 1.8 1.8) (drill 0.9) (layers *.Cu *.Mask)
+      (net 7 "Net-(BT1-Pad1)") (pinfunction "A") (pintype "passive"))
+    (pad "2" thru_hole circle (at 2.5 0) (size 1.8 1.8) (drill 0.9) (layers *.Cu *.Mask)
+      (net 2 "+3V3") (pinfunction "B") (pintype "passive"))
+    (pad "3" thru_hole circle (at 5 0) (size 1.8 1.8) (drill 0.9) (layers *.Cu *.Mask)
+      (net 8 "unconnected-(SW1-Pad3)") (pinfunction "C") (pintype "passive"))
+    (pad "4" thru_hole circle (at 0 6) (size 1.8 1.8) (drill 0.9) (layers *.Cu *.Mask)
+      (net 9 "unconnected-(SW1-Pad4)") (pinfunction "A") (pintype "passive"))
+    (pad "5" thru_hole circle (at 2.5 6) (size 1.8 1.8) (drill 0.9) (layers *.Cu *.Mask)
+      (net 10 "unconnected-(SW1-Pad5)") (pinfunction "B") (pintype "passive"))
+    (pad "6" thru_hole circle (at 5 6) (size 1.8 1.8) (drill 0.9) (layers *.Cu *.Mask)
+      (net 11 "unconnected-(SW1-Pad6)") (pinfunction "C") (pintype "passive"))
+    (model "${KICAD6_3DMODEL_DIR}/Button_Switch_THT.3dshapes/SW_Push_2P2T_Toggle_CK_PVA2xxH3xxxxxxV2.wrl"
       (offset (xyz 0 0 0))
       (scale (xyz 1 1 1))
@@
     (fp_arc (start 1.95 -5.5) (mid 27.78107 0) (end 1.95 5.5) (layer "B.Fab") (width 0.1))
     (pad "1" thru_hole rect locked (at 0 0) (size 2.1 2.1) (drill 1.3) (layers *.Cu *.Mask)
-      (net 2 "+3V3") (pinfunction "+") (pintype "passive"))
+      (net 7 "Net-(BT1-Pad1)") (pinfunction "+") (pintype "passive"))
     (pad "2" thru_hole circle locked (at 20 0) (size 2.1 2.1) (drill 1.3) (layers *.Cu *.Mask)
       (net 3 "GND") (pinfunction "-") (pintype "passive"))

Commit message: 21.06.2022
Parts:
- removed BT1: Battery_Cell, Battery2:BatteryHolder_ComfortableElectronic_CH273-2450_1x2450
- removed SW1: SW_Push_DPDT, Button_Switch_THT:SW_Push_2P2T_Toggle_CK_PVA2xxH3xxxxxxV2
- added BT?: Battery_Cell, Battery:BatteryHolder_ComfortableElectronic_CH273-2450_1x2450, F.Cu at (175.3, 91.4)
- added J?: AVR-ISP-6, Connector_PinHeader_2.54mm:PinHeader_2x03_P2.54mm_Vertical, F.Cu at (206.2, 89.2)
- added J?: Conn_01x03, Connector_PinSocket_2.54mm:PinSocket_1x03_P2.54mm_Vertical, F.Cu at (206.2, 79.5)
- added JP1: SolderJumper_2_Open, Jumper:SolderJumper-2_P1.3mm_Open_TrianglePad1.0x1.5mm, F.Cu at (160.0, 78.7)
- added JP?: SolderJumper_2_Open, Jumper:SolderJumper-2_P1.3mm_Open_TrianglePad1.0x1.5mm, F.Cu at (210.6, 78.9)
- added R?: 4.7K, Resistor_SMD:R_0805_2012Metric, F.Cu at (175.5, 107.2)
Connections:
- RF1 pad 1: Net-(RF1-Pad1) -> Net-(JP2-Pad2)
- U1 pad 1: Net-(RF1-Pad1) -> Net-(J2-Pad4)
- U1 pad 3: unconnected-(U1-Pad3) -> Net-(J2-Pad3)
- U1 pad 4: unconnected-(U1-Pad4) -> Net-(J1-Pad2)
- U1 pad 6: unconnected-(U1-Pad6) -> Net-(J2-Pad5)

Commit message: 01.07.2022
Parts:
- removed JP1, JP?: SolderJumper_2_Open, Jumper:SolderJumper-2_P1.3mm_Open_TrianglePad1.0x1.5mm
- added C1: 100n, Capacitor_SMD:C_0805_2012Metric, F.Cu at (185.7, 98.3)
- added D1: SFH4346, LED_THT:LED_D3.0mm, F.Cu at (193.0, 86.6)
- added J1: Conn_01x02, Connector_PinHeader_2.54mm:PinHeader_1x02_P2.54mm_Vertical, F.Cu at (190.0, 97.5)
- added J1: Conn_01x02, Connector_PinHeader_2.54mm:PinHeader_1x02_P2.54mm_Vertical, F.Cu at (179.8, 96.5)
- added J?: Conn_01x02, Connector_PinHeader_2.54mm:PinHeader_1x02_P2.54mm_Vertical, F.Cu at (196.6, 92.2)
- added R?: 4.7K, Resistor_SMD:R_0805_2012Metric, F.Cu at (187.0, 92.2)
- added R?: 4.7K, Resistor_SMD:R_0805_2012Metric, F.Cu at (190.2, 89.4)
- BT?: moved to B.Cu
- moved RF1 51.4 mm to (188.0, 81.3), turned to 180 degrees
- moved U1 42.0 mm to (185.7, 95.2)
- moved J? 30.3 mm to (185.4, 101.6), turned to 90 degrees
- moved J? 26.5 mm to (179.8, 86.1)
- moved BT? 19.8 mm to (188.0, 106.7), turned to 90 degrees
- moved R? 19.1 mm to (189.7, 94.5), turned to 180 degrees
Connections:
- J? pad 4: Net-(J2-Pad4) -> Net-(J4-Pad4)
- RF1 pad 1: Net-(JP2-Pad2) -> Net-(J4-Pad4)
- U1 pad 1: Net-(J2-Pad4) -> Net-(J4-Pad4)
Routing:
- net (no net): vias 0 -> 4
Other:
- board outline added: 30.2 x 39.6 mm

Commit message: 08.07.2022
Parts:
- removed the J? at (196.6, 92.2)
- removed the J? at (185.4, 101.6)
- added J3: Conn_01x03, Connector_PinHeader_2.54mm:PinHeader_1x03_P2.54mm_Vertical, F.Cu at (179.8, 103.4)
- added RF2: RF_Receiver_433_MHz, Connector_PinHeader_2.54mm:PinHeader_1x04_P2.54mm_Vertical, F.Cu at (190.5, 77.7)
- added SW1: SW_Push_Dual_x2, Button_Switch_THT:SW_PUSH_6mm_H4.3mm, F.Cu at (199.8, 95.5)
- moved J1 5.93 mm to (191.0, 103.4)
- moved R? 1.81 mm to (186.7, 90.4)
Routing:
- added copper zone on F.Cu, net GND
Other:
- board size 30.2 x 39.6 mm -> 30.3 x 35.9 mm
