File: 433 MHz/TX_tiny10/TX_tiny10.kicad_pcb (KiCad board)
At the start: 2 copper layers, 30.3 x 35.9 mm, 14 parts, among them J1 Conn_01x02, J3 Conn_01x03, SW1 SW_Push_Dual_x2, U1 ATtiny10-TS

Commit message: 12.07.2022
Parts:
- U1: footprint Package_TO_SOT_SMD:SOT-23-6 -> Package_TO_SOT_SMD:SOT-23-6_Handsoldering
- moved R? 0.25 mm to (190.0, 94.5)
Changed lines of the file:
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@@
   )
   (footprint "Resistor_SMD:R_0805_2012Metric" (layer "F.Cu")
-    (at 189.738 94.488 180)
+    (at 189.992 94.488 180)
     (descr "Resistor SMD 0805 (2012 Metric), square (rectangular) end terminal, IPC_7351 nominal, (Body size source: IPC-SM-782 page 72, https://www.pcb-3d.com/wordpress/wp-content/uploads/ipc-sm-782a_amendment_1_and_2.pdf), generated with kicad-footprint-generator")
     (tags "resistor")
@@
     )
   )
-  (footprint "Package_TO_SOT_SMD:SOT-23-6" (layer "F.Cu")
+  (footprint "Package_TO_SOT_SMD:SOT-23-6_Handsoldering" (layer "F.Cu")
     (at 185.674 95.25)
-    (descr "SOT, 6 Pin (https://www.jedec.org/sites/default/files/docs/Mo-178c.PDF variant AB), generated with kicad-footprint-generator ipc_gullwing_generator.py")
-    (tags "SOT TO_SOT_SMD")
+    (descr "6-pin SOT-23 package, Handsoldering")
+    (tags "SOT-23-6 Handsoldering")
     (property "Sheetfile" "TX_tiny10.kicad_sch")
     (property "Sheetname" "")
     (attr smd)
-    (fp_text reference "U1" (at -3.048 -1.016) (layer "F.SilkS")
+    (fp_text reference "U1" (at 0 -2.9) (layer "F.SilkS")
       (effects (font (size 1 1) (thickness 0.15)))
     )
-    (fp_text value "ATtiny10-TS" (at 0 2.4) (layer "F.Fab")
+    (fp_text value "ATtiny10-TS" (at 0 2.9) (layer "F.Fab")
       (effects (font (size 1 1) (thickness 0.15)))
     )
-    (fp_text user "${REFERENCE}" (at 0 0) (layer "F.Fab")
-      (effects (font (size 0.4 0.4) (thickness 0.06)))
+    (fp_text user "${REFERENCE}" (at 0 0 90) (layer "F.Fab")
+      (effects (font (size 0.5 0.5) (thickness 0.075)))
     )
-    (fp_line (start 0 1.56) (end 0.8 1.56) (layer "F.SilkS") (width 0.12))
-    (fp_line (start 0 -1.56) (end 0.8 -1.56) (layer "F.SilkS") (width 0.12))
-    (fp_line (start 0 1.56) (end -0.8 1.56) (layer "F.SilkS") (width 0.12))
-    (fp_line (start 0 -1.56) (end -1.8 -1.56) (layer "F.SilkS") (width 0.12))
-    (fp_line (start -2.05 1.7) (end 2.05 1.7) (layer "F.CrtYd") (width 0.05))
-    (fp_line (start -2.05 -1.7) (end -2.05 1.7) (layer "F.CrtYd") (width 0.05))
-    (fp_line (start 2.05 -1.7) (end -2.05 -1.7) (layer "F.CrtYd") (width 0.05))
-    (fp_line (start 2.05 1.7) (end 2.05 -1.7) (layer "F.CrtYd") (width 0.05))
-    (fp_line (start -0.8 -1.05) (end -0.4 -1.45) (layer "F.Fab") (width 0.1))
-    (fp_line (start -0.8 1.45) (end -0.8 -1.05) (layer "F.Fab") (width 0.1))
-    (fp_line (start 0.8 -1.45) (end 0.8 1.45) (layer "F.Fab") (width 0.1))
-    (fp_line (start -0.4 -1.45) (end 0.8 -1.45) (layer "F.Fab") (width 0.1))
-    (fp_line (start 0.8 1.45) (end -0.8 1.45) (layer "F.Fab") (width 0.1))
-    (pad "1" smd roundrect (at -1.1375 -0.95) (size 1.325 0.6) (layers "F.Cu" "F.Paste" "F.Mask") (roundrect_rratio 0.25)
+    (fp_line (start -0.9 1.61) (end 0.9 1.61) (layer "F.SilkS") (width 0.12))
+    (fp_line (start 0.9 -1.61) (end -2.05 -1.61) (layer "F.SilkS") (width 0.12))
+    (fp_line (start 2.4 -1.8) (end 2.4 1.8) (layer "F.CrtYd") (width 0.05))
+    (fp_line (start 2.4 1.8) (end -2.4 1.8) (layer "F.CrtYd") (width 0.05))
+    (fp_line (start -2.4 -1.8) (end 2.4 -1.8) (layer "F.CrtYd") (width 0.05))
+    (fp_line (start -2.4 1.8) (end -2.4 -1.8) (layer "F.CrtYd") (width 0.05))
+    (fp_line (start 0.9 -1.55) (end -0.25 -1.55) (layer "F.Fab") (width 0.1))
+    (fp_line (start -0.9 -0.9) (end -0.9 1.55) (layer "F.Fab") (width 0.1))
+    (fp_line (start 0.9 1.55) (end -0.9 1.55) (layer "F.Fab") (width 0.1))
+    (fp_line (start -0.9 -0.9) (end -0.25 -1.55) (layer "F.Fab") (width 0.1))
+    (fp_line (start 0.9 -1.55) (end 0.9 1.55) (layer "F.Fab") (width 0.1))
+    (pad "1" smd rect (at -1.35 -0.95) (size 1.56 0.65) (layers "F.Cu" "F.Paste" "F.Mask")
       (net 8 "Net-(J4-Pad4)") (pinfunction "PB0") (pintype "bidirectional"))
-    (pad "2" smd roundrect (at -1.1375 0) (size 1.325 0.6) (layers "F.Cu" "F.Paste" "F.Mask") (roundrect_rratio 0.25)
+    (pad "2" smd rect (at -1.35 0) (size 1.56 0.65) (layers "F.Cu" "F.Paste" "F.Mask")
       (net 2 "GND") (pinfunction "GND") (pintype "power_in"))
-    (pad "3" smd roundrect (at -1.1375 0.95) (size 1.325 0.6) (layers "F.Cu" "F.Paste" "F.Mask") (roundrect_rratio 0.25)
+    (pad "3" smd rect (at -1.35 0.95) (size 1.56 0.65) (layers "F.Cu" "F.Paste" "F.Mask")
       (net 7 "Net-(J4-Pad3)") (pinfunction "PB1") (pintype "bidirectional"))
-    (pad "4" smd roundrect (at 1.1375 0.95) (size 1.325 0.6) (layers "F.Cu" "F.Paste" "F.Mask") (roundrect_rratio 0.25)
+    (pad "4" smd rect (at 1.35 0.95) (size 1.56 0.65) (layers "F.Cu" "F.Paste" "F.Mask")
       (net 4 "Net-(J2-Pad1)") (pinfunction "PB2") (pintype "bidirectional"))
-    (pad "5" smd roundrect (at 1.1375 0) (size 1.325 0.6) (layers "F.Cu" "F.Paste" "F.Mask") (roundrect_rratio 0.25)
+    (pad "5" smd rect (at 1.35 0) (size 1.56 0.65) (layers "F.Cu" "F.Paste" "F.Mask")
       (net 1 "+3V3") (pinfunction "VCC") (pintype "power_in"))
-    (pad "6" smd roundrect (at 1.1375 -0.95) (size 1.325 0.6) (layers "F.Cu" "F.Paste" "F.Mask") (roundrect_rratio 0.25)
+    (pad "6" smd rect (at 1.35 -0.95) (size 1.56 0.65) (layers "F.Cu" "F.Paste" "F.Mask")
       (net 9 "Net-(J4-Pad5)") (pinfunction "~{RESET}/PB3") (pintype "bidirectional"))
     (model "${KICAD6_3DMODEL_DIR}/Package_TO_SOT_SMD.3dshapes/SOT-23-6.wrl"
