File: 433 MHz/TX_tiny10/TX_tiny10.kicad_sch (KiCad schematic)
At the start: 3 parts, among them U1 ATtiny10-TS

Commit message: 21.06.2022
Parts:
- added SW1: SW_Push_DPDT, Button_Switch_THT:SW_Push_2P2T_Toggle_CK_PVA2xxH3xxxxxxV2, symbol Switch:SW_Push_DPDT
Connections:
- net +3V3: now also SW1.2 (B); no longer BT1.1 (+)
- new net: BT1.1 (+), SW1.1 (A)
Changed lines of the file:
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@@
     (pin "1")
   )
-  (symbol (lib_id "power:+3V3") (at 173.99 82.55 0) (unit 1)
+  (symbol (lib_id "power:+3V3") (at 176.53 72.39 0) (unit 1)
     (in_bom yes) (on_board yes) (fields_autoplaced)
-    (property "Reference" "#PWR0106" (id 0) (at 173.99 86.36 0)
+    (property "Reference" "#PWR0106" (id 0) (at 176.53 76.2 0)
       (effects (font (size 1.27 1.27)) hide)
     )
-    (property "Value" "+3V3" (id 1) (at 173.99 77.47 0))
-    (property "Footprint" "" (id 2) (at 173.99 82.55 0)
+    (property "Value" "+3V3" (id 1) (at 176.53 67.31 0))
+    (property "Footprint" "" (id 2) (at 176.53 72.39 0)
       (effects (font (size 1.27 1.27)) hide)
     )
-    (property "Datasheet" "" (id 3) (at 173.99 82.55 0)
+    (property "Datasheet" "" (id 3) (at 176.53 72.39 0)
       (effects (font (size 1.27 1.27)) hide)
     )
@@
     (pin "1")
   )
+  (symbol (lib_id "Switch:SW_Push_DPDT") (at 181.61 77.47 90) (mirror x) (unit 1)
+    (in_bom yes) (on_board yes) (fields_autoplaced)
+    (property "Reference" "SW1" (id 0) (at 172.72 76.1999 90)
+      (effects (font (size 1.27 1.27)) (justify left))
+    )
+    (property "Value" "SW_Push_DPDT" (id 1) (at 172.72 78.7399 90)
+      (effects (font (size 1.27 1.27)) (justify left))
+    )
+    (property "Footprint" "Button_Switch_THT:SW_Push_2P2T_Toggle_CK_PVA2xxH3xxxxxxV2" (id 2) (at 176.53 77.47 0)
+      (effects (font (size 1.27 1.27)) hide)
+    )
+    (property "Datasheet" "~" (id 3) (at 176.53 77.47 0)
+      (effects (font (size 1.27 1.27)) hide)
+    )
+    (pin "1")
+    (pin "2")
+    (pin "3")
+    (pin "4")
+    (pin "5")
+    (pin "6")
+  )
   (sheet_instances
     (path "/" (page "1"))
@@
       (reference "RF1") (unit 1) (value "RF_Transmitter_433_MHz") (footprint "Sensors:RF_Transmitter_433_MHz")
     )
+    (path "/e0904428-9586-4daa-bae3-1cd482cc010a"
+      (reference "SW1") (unit 1) (value "SW_Push_DPDT") (footprint "Button_Switch_THT:SW_Push_2P2T_Toggle_CK_PVA2xxH3xxxxxxV2")
+    )
     (path "/97df36b4-64e2-41e3-92ff-44055cc5a9b6"

Commit message: 21.06.2022
Parts:
- removed SW1: SW_Push_DPDT, Button_Switch_THT:SW_Push_2P2T_Toggle_CK_PVA2xxH3xxxxxxV2, symbol Switch:SW_Push_DPDT
- added J1: Conn_01x03, Connector_PinHeader_2.54mm:PinHeader_1x03_P2.54mm_Vertical, symbol Connector_Generic:Conn_01x03
- added J2: AVR-ISP-6, Connector_PinHeader_2.54mm:PinHeader_2x03_P2.54mm_Vertical, symbol Connector:AVR-ISP-6
- added JP1, JP2: SolderJumper_2_Open, Jumper:SolderJumper-2_P1.3mm_Open_TrianglePad1.0x1.5mm, symbol Jumper:SolderJumper_2_Open
- added R1: 4.7K, Resistor_SMD:R_0805_2012Metric, symbol Device:R
Connections:
- net +3V3: now also BT1.1 (+), J1.1 (Pin_1), J2.2 (VCC), R1.2
- net GND: now also J1.3 (Pin_3), J2.6 (GND)
- net at U1.1 (PB0): now also J2.4 (MOSI), JP2.1 (A); no longer RF1.1 (DATA)
- net at U1.3 (PB1): now also J2.3 (SCK)
- net at U1.4 (PB2): now also J1.2 (Pin_2), JP1.2 (B)
- net at U1.6 (~{RESET}/PB3): now also J2.5 (~{RST})
- new net: JP1.1 (A), R1.1
- new net: JP2.2 (B), RF1.1 (DATA)

Commit message: 01.07.2022
Parts:
- removed JP1, JP2: SolderJumper_2_Open, Jumper:SolderJumper-2_P1.3mm_Open_TrianglePad1.0x1.5mm, symbol Jumper:SolderJumper_2_Open
- added C1: 100n, Capacitor_SMD:C_0805_2012Metric, symbol Device:C
- added D1: SFH4346, LED_THT:LED_D3.0mm, symbol LED:SFH4346
- added J1 (x2), J5: Conn_01x02, Connector_PinHeader_2.54mm:PinHeader_1x02_P2.54mm_Vertical, symbol Connector_Generic:Conn_01x02
- added R2, R3: 4.7K, Resistor_SMD:R_0805_2012Metric, symbol Device:R
- renumbered J1 to J3, J2 to J4
Connections:
- net +3V3: now also C1.1, J1.1 (Pin_1), R3.2
- net GND: now also C1.2, D1.1 (K), J1.2 (Pin_2), J5.2 (Pin_2)
- net at R1.1: now also J1.2 (Pin_2)
- net at J3.2 (Pin_2), U1.4 (PB2): now also J1.1 (Pin_1), J5.1 (Pin_1)
- net at J4.4 (MOSI), U1.1 (PB0): now also RF1.1 (DATA)
- net at J4.3 (SCK), U1.3 (PB1): now also R2.2
- net at J4.5 (~{RST}), U1.6 (~{RESET}/PB3): now also R3.1
- new net: D1.2 (A), R2.1
Other:
- moved on the sheet: R1, RF1

Commit message: 08.07.2022
Parts:
- removed J5: Conn_01x02, Connector_PinHeader_2.54mm:PinHeader_1x02_P2.54mm_Vertical, symbol Connector_Generic:Conn_01x02
- added RF2: RF_Receiver_433_MHz, Connector_PinHeader_2.54mm:PinHeader_1x04_P2.54mm_Vertical, symbol sensors:RF_Receiver_433_MHz
- added SW1: SW_Push_Dual_x2, Button_Switch_THT:SW_PUSH_6mm_H4.3mm, symbol Switch:SW_Push_Dual_x2
Connections:
- net +3V3: now also RF2.1 (VCC)
- net GND: now also RF2.4 (GND), SW1.2 (D)
- net at J1.1 (Pin_1), J3.2 (Pin_2), U1.4 (PB2): now also SW1.1 (C)
- net at J4.4 (MOSI), RF1.1 (DATA), U1.1 (PB0): now also RF2.2 (DATA)
Other:
- moved on the sheet: J1, R1

Commit message: 12.07.2022
Parts:
- U1: footprint Package_TO_SOT_SMD:SOT-23-6 -> Package_TO_SOT_SMD:SOT-23-6_Handsoldering
Changed lines of the file:
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@@
       (effects (font (size 1.27 1.27)) (justify right))
     )
-    (property "Footprint" "Package_TO_SOT_SMD:SOT-23-6" (id 2) (at 129.54 88.9 0)
+    (property "Footprint" "Package_TO_SOT_SMD:SOT-23-6_Handsoldering" (id 2) (at 129.54 88.9 0)
       (effects (font (size 1.27 1.27) italic) hide)
     )
@@
     )
     (path "/97df36b4-64e2-41e3-92ff-44055cc5a9b6"
-      (reference "U1") (unit 1) (value "ATtiny10-TS") (footprint "Package_TO_SOT_SMD:SOT-23-6")
-    )
-  )
+      (reference "U1") (unit 1) (value "ATtiny10-TS") (footprint "Package_TO_SOT_SMD:SOT-23-6_Handsoldering")
+    )
+  )
