File: 433 MHz/RXTX_tiny10/RXTX_tiny10.kicad_pcb (KiCad board)
At the start: 2 copper layers, 30.3 x 35.9 mm, 14 parts, among them J1 Conn_01x02, J3 Conn_01x03, SW1 SW_Push_Dual_x2, U1 ATtiny10-TS

Commit message: 13.07.2022
Parts:
- added G***: LOGO, LOGO, F.Cu at (192.0, 102.9)
- moved J1 15.6 mm to (176.0, 99.1)
- moved J1 11.1 mm to (176.0, 86.1)
- moved J3 8.98 mm to (176.0, 95.2)
- moved D1 4.64 mm to (197.6, 85.9)
- moved SW1 1.02 mm to (199.8, 94.5)
Other:
- board text added: "bs_kombo"

Commit message: 15.07.2022
Parts:
- added SW1: SW_DPDT_x2, Button_Switch_THT:SW_Slide_1P2T_CK_OS102011MS2Q, F.Cu at (175.5, 96.8)
- moved J1 6.86 mm to (180.3, 104.4)
- moved J3 6.65 mm to (180.3, 100.3), turned to 180 degrees
- moved G*** 4.91 mm to (196.6, 101.1)
- moved BT? 1.35 mm to (188.0, 105.3)
- moved RF1 0.36 mm to (188.2, 81.5)
- renumbered SW1 to SW2
Connections:
- BT? pad 1: +3V3 -> Net-(BT1-Pad1)
Routing:
- net +3V3: track 0.00 -> 56.9 mm
- net Net-(J2-Pad1): track 0.00 -> 37.1 mm
- net Net-(J4-Pad4): track 0.00 -> 22.8 mm
- net Net-(J4-Pad3): track 0.00 -> 22.1 mm
- net Net-(J2-Pad2): track 0.00 -> 21.2 mm
- net Net-(BT1-Pad1): track 0.00 -> 15.2 mm
- net Net-(J4-Pad5): track 0.00 -> 12.4 mm, vias 0 -> 1
- net Net-(D1-Pad2): track 0.00 -> 11.0 mm
- net GND: track 0.00 -> 2.59 mm, vias 0 -> 2
- added copper zone on B.Cu, net GND
Other:
- board text added: "+"
- board text added: "-"
- board text added: "MHXC"
- board text added: "data"
- board text added: "gnd"
- board text added: "in"
- board text added: "jumper"
- board text added: "vcc"
