File: 433 MHz/RXTX_tiny13/RXTX_tiny13.kicad_sch (KiCad schematic)
At the start: 15 parts, among them J1 Conn_01x02, J3 Conn_01x03, J4 AVR-ISP-6, SW1 SW_DPDT_x2, SW2 SW_Push_Dual_x2, U1 ATtiny10-TS

Commit message: 15.07.2022
Parts:
- removed U1: ATtiny10-TS, Package_TO_SOT_SMD:SOT-23-6_Handsoldering, symbol MCU_Microchip_ATtiny:ATtiny10-TS
- added U1: ATtiny13A-S, Package_SO:SOIC-8W_5.3x5.3mm_P1.27mm, symbol MCU_Microchip_ATtiny:ATtiny13A-S
Connections:
- net +3V3: now also U1.8 (VCC)
- net GND: now also U1.4 (GND)
- net at R2.2: no longer J4.3 (SCK)
- net at RF1.1 (DATA), RF2.2 (DATA): no longer J4.4 (MOSI)
- net at J4.5 (~{RST}): no longer R3.1
- new net: R3.1, U1.1 (~{RESET}/PB5)
Other:
- moved on the sheet: R3
